File: MainMCU.kicad_sch (KiCad schematic)
At the start: 9 parts, among them IC1 ESP32-WROOM-32E-N8, J5 20021121-00010C4LF, U4 NCP176AMX330TCG

Commit message: version 2 with 0.8mm thickness
Parts:
- removed U4: NCP176AMX330TCG, Library:XDFN6_711AT_ONS, symbol 2023-09-03_14-36-57:NCP176AMX330TCG
- added C5: 0.1u, Capacitor_SMD:C_0402_1005Metric, symbol Device:C
- added IC2: AP7366-33W5-7, Library:SOT95P285X130-5N, symbol 2023-09-03_14-36-57:AP7366-33W5-7
- added J3: 20021121-00006C4LF, Library:CONN_20021121-00006C4LF_AMP, symbol 2023-09-03_14-36-57:20021121-00006C4LF
Connections:
- net +3.3V: now also C5.1, C5.2, IC2.5 (OUT), J3.2; no longer C5.1
- net +BATT: now also C5.1, IC2.1 (IN), IC2.3 (EN); no longer C5.1
- net CH1_1: now also IC1.24 (IO2); no longer IC1.26 (IO4)
- net CH1_2: now also IC1.26 (IO4); no longer IC1.25 (IO0)
- net CH1_BTN: now also IC1.25 (IO0), J3.6; no longer IC1.24 (IO2)
- net EN: now also J3.1
- net GND: now also C5.1, IC2.2 (GND), J3.4
- net RXD: now reaches IC1.34 (RXD0)
- net RXD: now also J3.5
- net TXD: now reaches IC1.35 (TXD0)
- net TXD: now also J3.3
Other:
- note added: "IO0"
- note added: "TDI"
- moved on the sheet: C5, J5

Commit message: v3: removed digital potentiometer, added 8 discrete resistors and one GPIO expander
Connections:
- net +3.3V: now also J3.1; no longer J3.2
- net CH1_BTN: now also J3.5; no longer J3.6
- net EN: now also J3.2; no longer J3.1
- net GND: now also J3.3; no longer J3.4
- net RXD: now also J3.6; no longer J3.5
- net TXD: now also J3.4; no longer J3.3
- net CS renamed SCK

Commit message: version 4: changed GPIO expander, added current sense resistor to electrodes, added buzzer pins, fixed some gpio inputs that needs to be pulled high, added battery charge detection, added battery level measurement feature
Parts:
- added Q2: NPN, Package_TO_SOT_SMD:SOT-23, symbol Simulation_SPICE:NPN
- added R3 (x3): 1K, Resistor_SMD:R_0402_1005Metric, symbol Device:R
- C5: value DNP -> a
- IC2: Long Description (none) -> Linear Voltage Regulator IC Positive Fixed 1 Output 600mA S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
- J3: Long Description (none) -> Connector Header Surface Mount 6 position 0.050" (1.27mm)
- J5: Long Description (none) -> Connector Header Surface Mount 10 position 0.050" (1.27mm)
Connections:
- net +BATT: now also R3.2
- net GND: now also Q2.2 (E)
- net MISO renamed BAT_LEVEL
- net MODE_BTN renamed BUZZER_MCU
- net BUZZER_MCU: now also R3.2
- net OK_BTN renamed EL2_DET
- net SCLK renamed INT_IO_EXP
- net TIMER_BTN renamed EL1_DET
- new net: Q2.1 (B), R3.1
- new net BUZZER_N: Q2.3 (C), R3.1
- new net BUZZER_P: R3.1, R3.2
